File: hw/stm32g0/ir_receiver.kicad_sch (KiCad schematic)
At the start: 5 parts, among them U301 VS1838B

Commit message: chore(hw): update title blocks
Other:
- company: (none) -> Stefan Misik
- title: (none) -> STM32G0 LED Controller
Changed lines of the file:
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@@
 	(generator_version "8.0")
 	(paper "A4")
+	(title_block
+		(title "STM32G0 LED Controller")
+		(date "2024-06-29")
+		(company "Stefan Misik")
+		(comment 1 "www.stefanmisik.com")
+	)
 	(junction
 		(at 162.56 93.98)
